File: HoloCubic.sch (EAGLE design)
At the start: 2 parts, among them IC1 CP2102

Commit message: .
Parts:
- removed IC1: CP2102, common:CP2102
- removed U$1: LP2992, common:LP2992
- added C1: 0.1uF, rcl:C-EUC0402
- added C2: 10uF, rcl:C-EUC0402
- added C3: 10nF, rcl:C-EUC0402
- added R1: 10K, rcl:R-EU_R0402
- added R3: 200R, rcl:R-EU_R0402
- added R4, R5: 12K, rcl:R-EU_R0402
- added U1: LP2992, common:LP2992
- added U2: CP2102, common:CP2102
- added U3: (no value), common:ESP32-PICO
- added U4: (no value), common:MPU6050
- added USB1: TYPE-C-16PIN, usb:TYPE-C-16PIN
- added VT1, VT2: (no value), transistor:BC808-NPN-SOT23-BEC
Connections:
- new net +3V3: C1.1, C2.1, U1.VOUT
- new net +5V: R1.2, U1.ON/OFF, U1.VIN, U2.REGIN, U2.VBUS
- new net CP_RX: U2.RXD
- new net CP_TX: R3.2
- new net DTR: R4.2, U2.DTR, VT2.E
- new net EN: VT1.C
- new net GND: C1.2, C2.2, C3.2, U1.GND, U2.GND
- new net GPIO0: VT2.C
- new net N$1: C3.1, U1.BYPASS
- new net N$2: R1.1, U2.!RST
- new net N$3: R4.1, VT1.B
- new net N$4: R5.1, VT2.B
- new net N$5: R3.1, U2.TXD
- new net RTS: R5.2, U2.RTS, VT1.E
- new net USB-PWR-DM: U2.D-
- new net USB-PWR-DP: U2.D+
Other:
- note added: "POWER"
- note added: "USB-PROG"

Commit message: .
Parts:
- added C10, C11, C8: 0.1uF, rcl:C-EUC0402
- added C6: 10nF, rcl:C-EUC0402
- added C9: 2.2nF, rcl:C-EUC0402
- added CON1: (no value), common:FPC-0.5MM-8P
- added D1: WS2812B, common:WS2812B
- added J1: 0473521001, common:0473521001
- added R10, R11, R7, R8, R9: 10K, rcl:R-EU_R0402
- added U5: BH1750FVI-TR, common:BH1750FVI-TR
Connections:
- new net BH_SCL: U5.SCL
- new net BH_SDA: U5.SDA
- new net N$10: R11.1, U5.DVI
- new net N$6: U4.SDA
- new net N$7: U4.SCL
- new net N$8: C9.1, U4.CPOUT
- new net N$9: C8.2, U4.REGOTU
- new net REG_LED: D1.DI
- new net SD_CLK: J1.CLK, R9.1
- new net SD_CS: J1.CD/DATA3, R10.1
- new net SD_MISO: J1.DATA0, R7.1
- new net SD_MOSI: J1.CMD, R8.1
- net +3V3: now also C10.2, C6.2, J1.VDD, R10.2, R11.2, R7.2, R8.2, R9.2, U4.VDD, U4.VLOGIC
- net +5V: now also C11.2, D1.VDD, U5.VCC, USB1.A4, USB1.A9, USB1.B4, USB1.B9
- net GND: now also C10.1, C11.1, C6.1, C8.1, C9.2, D1.GND, J1.VSS, U4.AD0, U4.CLKIN, U4.FSYNC, U4.GND, U5.ADDR, U5.GND, USB1.A1, USB1.A12, USB1.B1, USB1.B12
- net USB-PWR-DM: now also USB1.A7, USB1.B7
- net USB-PWR-DP: now also USB1.A6, USB1.B6
Other:
- moved on the sheet: U3, U4
